Commit message: stuff?

File: ur_description/urdf/ur5_robot_with_gripper.urdf.xacro (robot description, xacro)
@@ -7,5 +7,5 @@
   <xacro:include filename="$(find ur_description)/urdf/ur5_with_gripper.urdf.xacro" />
   <!-- arm -->
-  <xacro:ur5_robot prefix="" joint_limited="false"/>
+  <xacro:ur5_robot prefix="" joint_limited="true"/>
   <link name="world" />
   <joint name="world_joint" type="fixed">

File: ur_description/urdf/ur5_with_gripper.urdf (robot description, URDF)
Before this commit: robot ur5, 25 links, 24 joints
Joints:
- joint elbow_joint: limit lower=-6.2831853 upper=6.2831853 effort=150.0 velocity=3.15 -> lower=-3.14159265 upper=3.14159265 effort=150.0 velocity=3.15
- joint shoulder_lift_joint: limit lower=-6.2831853 upper=6.2831853 effort=150.0 velocity=3.15 -> lower=-3.14159265 upper=3.14159265 effort=150.0 velocity=3.15
- joint shoulder_pan_joint: limit lower=-6.2831853 upper=6.2831853 effort=150.0 velocity=3.15 -> lower=-3.14159265 upper=3.14159265 effort=150.0 velocity=3.15
- joint world_joint: origin xyz=0.0 0.0 0.0 rpy=0.0 0.0 0.0 -> xyz=0.0 0.0 0.01 rpy=0.0 0.0 0.7853981633974483
- joint wrist_1_joint: limit lower=-6.2831853 upper=6.2831853 effort=28.0 velocity=3.2 -> lower=-3.14159265 upper=3.14159265 effort=28.0 velocity=3.2
- joint wrist_2_joint: limit lower=-6.2831853 upper=6.2831853 effort=28.0 velocity=3.2 -> lower=-3.14159265 upper=3.14159265 effort=28.0 velocity=3.2
- joint wrist_3_joint: limit lower=-6.2831853 upper=6.2831853 effort=28.0 velocity=3.2 -> lower=-3.14159265 upper=3.14159265 effort=28.0 velocity=3.2
